File: breakout-ttgf0p2-cob.kicad_pcb (KiCad board)
At the start: 4 copper layers, 50 x 50 mm, 77 parts, among them J1 Conn_01x12, J2 DF12NB-60DS-0.5V_51, J3 DF12NB-50DS-0.5V_51, U1 AP2112K-3.3, U2 AP2112K-3.3, U3 TT_GF_0p2_ASIC, U4 24LC02

Commit message: add wiring
Parts:
- removed the STITCH01 at (160.2, 93.5)
- removed the STITCH18 at (162.0, 86.9)
- removed the STITCHSM01 at (148.6, 56.4)
- added ?: , , F.Cu at (154.2, 75.2)
- added ?: , , F.Cu at (151.8, 65.2)
- added ?: , , F.Cu at (156.8, 62.8)
- added ?: , , F.Cu at (119.2, 95.2)
- added ?: , , F.Cu at (150.5, 84.0)
- added ?: , , F.Cu at (129.2, 95.2)
- added ?: , , F.Cu at (139.2, 95.2)
- added ?: , , F.Cu at (149.2, 72.8)
- added ?: , , F.Cu at (119.2, 82.8)
- added ?: , , F.Cu at (118.0, 59.0)
- added ?: , , F.Cu at (156.8, 72.8)
- added ?: , , F.Cu at (156.8, 67.8)
- added ?: , , F.Cu at (146.8, 67.8)
- added ?: , , F.Cu at (151.8, 92.8)
- added ?: , , F.Cu at (146.8, 63.0)
- added ?: , , F.Cu at (129.2, 87.8)
- added ?: , , F.Cu at (151.8, 70.2)
- added ?: , , F.Cu at (144.2, 85.2)
- added ?: , , F.Cu at (129.2, 55.5)
- added ?: , , F.Cu at (121.8, 60.2)
- added ?: , , F.Cu at (134.2, 90.2)
- added ?: , , F.Cu at (124.2, 80.2)
- added ?: , , F.Cu at (139.2, 87.8)
- added ?: , , F.Cu at (119.2, 87.8)
- added ?: , , F.Cu at (124.2, 85.2)
- added ?: , , F.Cu at (134.2, 58.0)
- added ?: , , F.Cu at (124.2, 90.2)
- added ?: , , F.Cu at (151.8, 57.8)
- added ?: , , F.Cu at (146.8, 90.2)
- added ?: , , F.Cu at (139.2, 60.2)
- added ?: , , F.Cu at (126.8, 60.2)
- moved R11 17.1 mm to (145.6, 55.7), turned to -90 degrees
- moved R10 10.1 mm to (148.1, 55.7), turned to -90 degrees
- moved TTLOGO1 8.87 mm to (151.8, 62.5)
- moved TP3 1.81 mm to (116.0, 61.9)
- moved C11 1.08 mm to (142.0, 66.4)
- moved C12 1.08 mm to (133.8, 66.4)
- moved C13 1.08 mm to (135.2, 66.4)
- moved C17 1.08 mm to (138.6, 66.2)
- moved C14 0.69 mm to (141.7, 81.1)
- moved C10 0.59 mm to (134.8, 80.9)
- moved C16 0.59 mm to (138.0, 81.1)
Routing:
- net GND: track 67.2 -> 114.0 mm, vias 24 -> 87
- net /increment: track 1.75 -> 48.6 mm, vias 0 -> 1
- net VDD_{IO}: track 47.4 -> 94.2 mm, vias 6 -> 7
- net /rst_n: track 1.99 -> 45.9 mm, vias 0 -> 2
- net /an21: track 0.00 -> 30.5 mm, vias 0 -> 1
- net /an20: track 0.00 -> 29.8 mm, vias 0 -> 1
- net /an19: track 0.00 -> 28.6 mm, vias 0 -> 1
- net /enable: track 33.4 -> 61.4 mm, vias 2 -> 1
- net /an18: track 0.00 -> 27.8 mm, vias 0 -> 1
- net /an0: track 0.00 -> 27.6 mm, vias 0 -> 1
- net /an1: track 0.00 -> 27.0 mm, vias 0 -> 1
- net /an17: track 0.00 -> 27.0 mm, vias 0 -> 1
- net /an2: track 0.00 -> 26.4 mm, vias 0 -> 1
- net /an16: track 0.00 -> 26.3 mm, vias 0 -> 1
- net /an3: track 0.00 -> 26.0 mm, vias 0 -> 1
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Other:
- board text removed: "ASIC"
- board text removed: "COB breakout"
- board text removed: "v${REVISION}"
